File: Hardware_Solder_3.3/Hardware_Solder_3.3.1.kicad_sch (KiCad schematic)
At the start: 95 parts, among them J1 Connector, J2 POWER, J3 SENSOR, J4 BATTERY, J5 Control Panel, J6 SWD DEBUG, J7 HEAT_WIRE, Q1 S8050, Q2 S8050, Q3 S8550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

Commit message: Add files via upload
Parts:
- J4: footprint Connector_PinHeader_2.54mm:PinHeader_2x01_P2.54mm_Vertical -> Connector_PinHeader_2.54mm:PinHeader_1x02_P2.54mm_Vertical_SMD_Pin1Right
Connections:
- net PWM: now also J5.1 (Pin_1)
- net PWM LED: no longer names the net of U6.32 (PA11)
- net PWM LED: no longer J5.1 (Pin_1)
- no-connect marks 4 -> 5
Changed lines of the file:
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@@
   (junction (at 124.46 77.47) (diameter 0) (color 0 0 0 0)
   )
+  (no_connect (at 257.81 119.38))
   (no_connect (at 224.79 111.76))
   (no_connect (at 224.79 114.3))
@@
     (effects (font (size 1.8 1.8) (thickness 0.36) bold) (justify left bottom))
   )
-  (global_label "PWM LED" (shape bidirectional) (at 176.53 132.08 0) (fields_autoplaced)
-    (effects (font (size 1.27 1.27)) (justify left))
-    (property "Intersheet References" "${INTERSHEET_REFS}" (id 0) (at 187.5307 132.0006 0)
-      (effects (font (size 1.27 1.27)) (justify left) hide)
-    )
-  )
   (global_label "O_SPK" (shape bidirectional) (at 148.59 171.45 0) (fields_autoplaced)
     (effects (font (size 1.27 1.27)) (justify left))
@@
     )
   )
-  (global_label "PWM LED" (shape bidirectional) (at 257.81 119.38 0) (fields_autoplaced)
-    (effects (font (size 1.27 1.27)) (justify left))
-    (property "Intersheet References" "${INTERSHEET_REFS}" (id 0) (at 268.8107 119.3006 0)
-      (effects (font (size 1.27 1.27)) (justify left) hide)
-    )
-  )
   (global_label "ESP_Tx" (shape bidirectional) (at 224.79 119.38 180) (fields_autoplaced)
     (effects (font (size 1.27 1.27)) (justify right))
@@
     )
   )
+  (global_label "PWM" (shape bidirectional) (at 176.53 132.08 0) (fields_autoplaced)
+    (effects (font (size 1.27 1.27)) (justify left))
+    (property "Intersheet References" "${INTERSHEET_REFS}" (id 0) (at 183.116 132.0006 0)
+      (effects (font (size 1.27 1.27)) (justify left) hide)
+    )
+  )
   (global_label "SWDIO" (shape bidirectional) (at 148.59 111.76 0) (fields_autoplaced)
     (effects (font (size 1.27 1.27)) (justify left))
@@
     (property "Reference" "J4" (id 0) (at 142.24 152.4 0))
     (property "Value" "BATTERY" (id 1) (at 147.32 149.86 0))
-    (property "Footprint" "Connector_PinHeader_2.54mm:PinHeader_2x01_P2.54mm_Vertical" (id 2) (at 143.51 152.4 0)
+    (property "Footprint" "Connector_PinHeader_2.54mm:PinHeader_1x02_P2.54mm_Vertical_SMD_Pin1Right" (id 2) (at 143.51 152.4 0)
       (effects (font (size 1.27 1.27)) hide)
     )
@@
     )
     (path "/9f5a1951-7c3a-48b2-a1da-6de70fa89839"
-      (reference "J4") (unit 1) (value "BATTERY") (footprint "Connector_PinHeader_2.54mm:PinHeader_2x01_P2.54mm_Vertical")
+      (reference "J4") (unit 1) (value "BATTERY") (footprint "Connector_PinHeader_2.54mm:PinHeader_1x02_P2.54mm_Vertical_SMD_Pin1Right")
     )
     (path "/f76ebf84-45ac-4e96-b2bd-85ec413e8fd9"
